File: Hardware/RackDistribution-4U/LightPanel.kicad_pcb (KiCad board)
At the start: 2 copper layers, 86.4 x 91.4 mm, 25 parts, among them J1 BoardToBoard

Commit message: Add libraries, 3d models and other bits
Other:
- board text added: "Tirga"
- board text removed: "--Tirga"
Changed lines of the file:
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@@
 			)
 		)
-		(property "Datasheet" "https://cdn-shop.adafruit.com/datasheets/WS2812B.pdf"
+		(property "Datasheet" "https://www.lcsc.com/datasheet/C52917433.pdf"
 			(at 0 0 180)
 			(unlocked yes)
@@
 			)
 		)
+		(property "LCSC#" "C52917433"
+			(at 0 0 180)
+			(unlocked yes)
+			(layer "F.Fab")
+			(hide yes)
+			(effects
+				(font
+					(size 1 1)
+					(thickness 0.15)
+				)
+			)
+		)
 		(property ki_fp_filters "LED*WS2812*PLCC*5.0x5.0mm*P3.2mm*")
 		(sheetname "/")
@@
 			)
 		)
-		(property "Datasheet" "https://cdn-shop.adafruit.com/datasheets/WS2812B.pdf"
+		(property "Datasheet" "https://www.lcsc.com/datasheet/C52917433.pdf"
 			(at 0 0 180)
 			(unlocked yes)
@@
 			)
 		)
+		(property "LCSC#" "C52917433"
+			(at 0 0 180)
+			(unlocked yes)
+			(layer "F.Fab")
+			(hide yes)
+			(effects
+				(font
+					(size 1 1)
+					(thickness 0.15)
+				)
+			)
+		)
 		(property ki_fp_filters "LED*WS2812*PLCC*5.0x5.0mm*P3.2mm*")
 		(sheetname "/")
@@
 			)
 		)
-		(property "Datasheet" "https://cdn-shop.adafruit.com/datasheets/WS2812B.pdf"
+		(property "Datasheet" "https://www.lcsc.com/datasheet/C52917433.pdf"
 			(at 0 0 180)
 			(unlocked yes)
@@
 			)
 		)
+		(property "LCSC#" "C52917433"
+			(at 0 0 180)
+			(unlocked yes)
+			(layer "F.Fab")
+			(hide yes)
+			(effects
+				(font
+					(size 1 1)
+					(thickness 0.15)
+				)
+			)
+		)
 		(property ki_fp_filters "LED*WS2812*PLCC*5.0x5.0mm*P3.2mm*")
 		(sheetname "/")
@@
 			)
 		)
-		(property "Datasheet" "https://cdn-shop.adafruit.com/datasheets/WS2812B.pdf"
+		(property "Datasheet" "https://www.lcsc.com/datasheet/C52917433.pdf"
 			(at 0 0 180)
 			(unlocked yes)
@@
 			)
 		)
+		(property "LCSC#" "C52917433"
+			(at 0 0 180)
+			(unlocked yes)
+			(layer "F.Fab")
+			(hide yes)
+			(effects
+				(font
+					(size 1 1)
+					(thickness 0.15)
+				)
+			)
+		)
 		(property ki_fp_filters "LED*WS2812*PLCC*5.0x5.0mm*P3.2mm*")
 		(sheetname "/")
@@
 			)
 		)
-		(property "Datasheet" "https://cdn-shop.adafruit.com/datasheets/WS2812B.pdf"
+		(property "Datasheet" "https://www.lcsc.com/datasheet/C52917433.pdf"
 			(at 0 0 180)
 			(unlocked yes)
@@
 			)
 		)
+		(property "LCSC#" "C52917433"
+			(at 0 0 180)
+			(unlocked yes)
+			(layer "F.Fab")
+			(hide yes)
+			(effects
+				(font
+					(size 1 1)
+					(thickness 0.15)
+				)
+			)
+		)
 		(property ki_fp_filters "LED*WS2812*PLCC*5.0x5.0mm*P3.2mm*")
 		(sheetname "/")
@@
 			)
 		)
-		(property "Datasheet" "https://cdn-shop.adafruit.com/datasheets/WS2812B.pdf"
+		(property "Datasheet" "https://www.lcsc.com/datasheet/C52917433.pdf"
 			(at 0 0 180)
 			(unlocked yes)
@@
 			)
 		)
+		(property "LCSC#" "C52917433"
+			(at 0 0 180)
+			(unlocked yes)
+			(layer "F.Fab")
+			(hide yes)
+			(effects
+				(font
+					(size 1 1)
+					(thickness 0.15)
+				)
+			)
+		)
 		(property ki_fp_filters "LED*WS2812*PLCC*5.0x5.0mm*P3.2mm*")
 		(sheetname "/")
@@
 			)
 		)
-		(property "Datasheet" "https://cdn-shop.adafruit.com/datasheets/WS2812B.pdf"
+		(property "Datasheet" "https://www.lcsc.com/datasheet/C52917433.pdf"
 			(at 0 0 180)
 			(unlocked yes)
@@
 			)
 		)
+		(property "LCSC#" "C52917433"
+			(at 0 0 180)
+			(unlocked yes)
+			(layer "F.Fab")
+			(hide yes)
+			(effects
+				(font
+					(size 1 1)
+					(thickness 0.15)
+				)
+			)
+		)
 		(property ki_fp_filters "LED*WS2812*PLCC*5.0x5.0mm*P3.2mm*")
 		(sheetname "/")
@@
 			)
 		)
-		(property "Datasheet" "https://cdn-shop.adafruit.com/datasheets/WS2812B.pdf"
+		(property "Datasheet" "https://www.lcsc.com/datasheet/C52917433.pdf"
 			(at 0 0 180)
 			(unlocked yes)
@@
 			)
 		)
+		(property "LCSC#" "C52917433"
+			(at 0 0 180)
+			(unlocked yes)
+			(layer "F.Fab")
+			(hide yes)
+			(effects
+				(font
+					(size 1 1)
+					(thickness 0.15)
+				)
+			)
+		)
 		(property ki_fp_filters "LED*WS2812*PLCC*5.0x5.0mm*P3.2mm*")
 		(sheetname "/")
@@
 			)
 		)
-		(property "Datasheet" "https://cdn-shop.adafruit.com/datasheets/WS2812B.pdf"
+		(property "Datasheet" "https://www.lcsc.com/datasheet/C52917433.pdf"
 			(at 0 0 180)
 			(unlocked yes)
@@
 			)
 		)
+		(property "LCSC#" "C52917433"
+			(at 0 0 180)
+			(unlocked yes)
+			(layer "F.Fab")
+			(hide yes)
+			(effects
+				(font
+					(size 1 1)
+					(thickness 0.15)
+				)
+			)
+		)
 		(property ki_fp_filters "LED*WS2812*PLCC*5.0x5.0mm*P3.2mm*")
 		(sheetname "/")
@@
 			)
 		)
-		(property "Datasheet" "https://cdn-shop.adafruit.com/datasheets/WS2812B.pdf"
+		(property "Datasheet" "https://www.lcsc.com/datasheet/C52917433.pdf"
 			(at 0 0 180)
 			(unlocked yes)
@@
 			)
 		)
+		(property "LCSC#" "C52917433"
+			(at 0 0 180)
+			(unlocked yes)
+			(layer "F.Fab")
+			(hide yes)
+			(effects
+				(font
+					(size 1 1)
+					(thickness 0.15)
+				)
+			)
+		)
 		(property ki_fp_filters "LED*WS2812*PLCC*5.0x5.0mm*P3.2mm*")
 		(sheetname "/")
@@
 			)
 		)
-		(model "/home/joe/Documents/3D Modeling/Lithium Water Cooling Parts/WaterCoolingRack-Body.step"
+		(model "${KIPRJMOD}/Libraries/project/3d/WaterCoolingRack-Light Gaurd.step"
 			(offset
 				(xyz -25.5 38 0)
@@
 			)
 			(rotate
-				(xyz 90 -0 -0)
+				(xyz 90 -0 -180)
 			)
 		)
@@
 			)
 		)
-		(property "Datasheet" "https://cdn-shop.adafruit.com/datasheets/WS2812B.pdf"
+		(property "Datasheet" "https://www.lcsc.com/datasheet/C52917433.pdf"
 			(at 0 0 180)
 			(unlocked yes)
@@
 			)
 		)
+		(property "LCSC#" "C52917433"
+			(at 0 0 180)
+			(unlocked yes)
+			(layer "F.Fab")
+			(hide yes)
+			(effects
+				(font
+					(size 1 1)
+					(thickness 0.15)
+				)
+			)
+		)
 		(property ki_fp_filters "LED*WS2812*PLCC*5.0x5.0mm*P3.2mm*")
 		(sheetname "/")
@@
 			)
 		)
-		(property "Datasheet" "https://cdn-shop.adafruit.com/datasheets/WS2812B.pdf"
+		(property "Datasheet" "https://www.lcsc.com/datasheet/C52917433.pdf"
 			(at 0 0 180)
 			(unlocked yes)
@@
 			)
 		)
+		(property "LCSC#" "C52917433"
+			(at 0 0 180)
+			(unlocked yes)
+			(layer "F.Fab")
+			(hide yes)
+			(effects
+				(font
+					(size 1 1)
+					(thickness 0.15)
+				)
+			)
+		)
 		(property ki_fp_filters "LED*WS2812*PLCC*5.0x5.0mm*P3.2mm*")
 		(sheetname "/")
@@
 			)
 		)
-		(property "Datasheet" "https://cdn-shop.adafruit.com/datasheets/WS2812B.pdf"
+		(property "Datasheet" "https://www.lcsc.com/datasheet/C52917433.pdf"
 			(at 0 0 180)
 			(unlocked yes)
@@
 			)
 		)
+		(property "LCSC#" "C52917433"
+			(at 0 0 180)
+			(unlocked yes)
+			(layer "F.Fab")
+			(hide yes)
+			(effects
+				(font
+					(size 1 1)
+					(thickness 0.15)
+				)
+			)
+		)
 		(property ki_fp_filters "LED*WS2812*PLCC*5.0x5.0mm*P3.2mm*")
 		(sheetname "/")
@@
 			)
 		)
-		(property "Datasheet" "https://cdn-shop.adafruit.com/datasheets/WS2812B.pdf"
+		(property "Datasheet" "https://www.lcsc.com/datasheet/C52917433.pdf"
 			(at 0 0 180)
 			(unlocked yes)
@@
 			)
 		)
+		(property "LCSC#" "C52917433"
+			(at 0 0 180)
+			(unlocked yes)
+			(layer "F.Fab")
+			(hide yes)
+			(effects
+				(font
+					(size 1 1)
+					(thickness 0.15)
+				)
+			)
+		)
 		(property ki_fp_filters "LED*WS2812*PLCC*5.0x5.0mm*P3.2mm*")
 		(sheetname "/")
@@
 			)
 		)
-		(property "Datasheet" "https://cdn-shop.adafruit.com/datasheets/WS2812B.pdf"
+		(property "Datasheet" "https://www.lcsc.com/datasheet/C52917433.pdf"
 			(at 0 0 180)
 			(unlocked yes)
@@
 			)
 		)
+		(property "LCSC#" "C52917433"
+			(at 0 0 180)
+			(unlocked yes)
+			(layer "F.Fab")
+			(hide yes)
+			(effects
+				(font
+					(size 1 1)
+					(thickness 0.15)
+				)
+			)
+		)
 		(property ki_fp_filters "LED*WS2812*PLCC*5.0x5.0mm*P3.2mm*")
 		(sheetname "/")
@@
 			)
 		)
-		(property "Datasheet" "https://cdn-shop.adafruit.com/datasheets/WS2812B.pdf"
+		(property "Datasheet" "https://www.lcsc.com/datasheet/C52917433.pdf"
 			(at 0 0 180)
 			(unlocked yes)
@@
 			)
 		)
+		(property "LCSC#" "C52917433"
+			(at 0 0 180)
+			(unlocked yes)
+			(layer "F.Fab")
+			(hide yes)
+			(effects
+				(font
+					(size 1 1)
+					(thickness 0.15)
+				)
+			)
+		)
 		(property ki_fp_filters "LED*WS2812*PLCC*5.0x5.0mm*P3.2mm*")
 		(sheetname "/")
@@
 		(layer "Edge.Cuts")
 	)
-	(gr_text "--Tirga"
-		(at 154.715 132.29 0)
+	(gr_text "Tirga"
+		(at 141 132.29 0)
 		(layer "B.SilkS")
 		(effects
@@
 				(bold yes)
 			)
-			(justify left bottom mirror)
+			(justify top mirror)
 		)
 	)
