File: Hardware/LightPanel/LightPanel.kicad_pcb (KiCad board)
At the start: 2 copper layers, 86.4 x 91.4 mm, 25 parts, among them J1 BoardToBoard

Commit message: Fix DRC
Parts:
- moved G*** 31.7 mm to (142.5, 90.0)
- moved REF** 31.7 mm to (136.3, 99.5)
- moved REF** 31.7 mm to (131.3, 91.8)
- moved G*** 11.5 mm to (132.0, 121.5)
Changed lines of the file:
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@@
 		(property "Reference" "H4"
 			(at 0 -5.25 0)
-			(layer "F.SilkS")
+			(layer "F.Fab")
 			(effects
 				(font
@@
 		(property "Reference" "H3"
 			(at 0 -5.25 0)
-			(layer "F.SilkS")
+			(layer "F.Fab")
 			(effects
 				(font
@@
 		(property "Reference" "H1"
 			(at 0 -5.25 0)
-			(layer "F.SilkS")
+			(layer "F.Fab")
 			(effects
 				(font
@@
 		(property "Reference" "H2"
 			(at 0 -5.25 0)
-			(layer "F.SilkS")
+			(layer "F.Fab")
 			(effects
 				(font
@@
 	(footprint "KenwoodFox:KITSUNE_LOGO"
 		(layer "B.Cu")
-		(at 123 115 180)
+		(at 142.5 90 180)
 		(property "Reference" "G***"
 			(at 0 0 0)
@@
 	(footprint "Symbol:OSHW-Logo2_9.8x8mm_SilkScreen"
 		(layer "B.Cu")
-		(at 111.76 116.84 180)
+		(at 131.26 91.84 180)
 		(descr "Open Source Hardware Symbol")
 		(tags "Logo Symbol OSHW")
@@
 	(footprint "Symbol:KiCad-Logo2_8mm_SilkScreen"
 		(layer "B.Cu")
-		(at 116.84 124.46 180)
+		(at 136.34 99.46 180)
 		(descr "KiCad Logo")
 		(tags "Logo KiCad")
@@
 	(footprint "Tirga:TirgaBrain"
 		(layer "B.Cu")
-		(at 143.51 121.92 180)
+		(at 132 121.5 180)
 		(property "Reference" "G***"
 			(at 0 0 0)
@@
 	)
 	(gr_text "I do not think\ntherefore\nI do not am."
-		(at 172.72 129.54 -0)
+		(at 161.21 129.12 -0)
 		(layer "B.SilkS")
 		(effects
@@
 	)
 	(barcode
-		(at 115 100.5 0)
+		(at 117 95.5 0)
 		(layer "B.SilkS")
 		(size 15 15)
@@
 		(at 121.666 81.28)
 		(size 0.8)
-		(drill 0.7)
+		(drill 0.6)
 		(layers "F.Cu" "B.Cu")
 		(net "+5V")
@@
 		(at 134.62 55.372)
 		(size 0.8)
-		(drill 0.7)
+		(drill 0.6)
 		(layers "F.Cu" "B.Cu")
 		(net "+5V")
@@
 		(at 159.512 131.826)
 		(size 0.8)
-		(drill 0.7)
+		(drill 0.6)
 		(layers "F.Cu" "B.Cu")
 		(net "+5V")
@@
 		(at 134.112 81.026)
 		(size 0.8)
-		(drill 0.7)
+		(drill 0.6)
 		(layers "F.Cu" "B.Cu")
 		(net "+5V")
@@
 		(at 121.666 106.426)
 		(size 0.8)
-		(drill 0.7)
+		(drill 0.6)
 		(layers "F.Cu" "B.Cu")
 		(net "+5V")
@@
 		(at 159.766 106.68)
 		(size 0.8)
-		(drill 0.7)
+		(drill 0.6)
 		(layers "F.Cu" "B.Cu")
 		(net "+5V")
@@
 		(at 121.666 132.08)
 		(size 0.8)
-		(drill 0.7)
+		(drill 0.6)
 		(layers "F.Cu" "B.Cu")
 		(net "+5V")
@@
 		(at 172.466 106.68)
 		(size 0.8)
-		(drill 0.7)
+		(drill 0.6)
 		(layers "F.Cu" "B.Cu")
 		(net "+5V")
@@
 		(at 172.466 131.826)
 		(size 0.8)
-		(drill 0.7)
+		(drill 0.6)
 		(layers "F.Cu" "B.Cu")
 		(net "+5V")
@@
 		(at 171.958 80.772)
 		(size 0.8)
-		(drill 0.7)
+		(drill 0.6)
 		(layers "F.Cu" "B.Cu")
 		(net "+5V")
@@
 		(at 134.62 131.826)
 		(size 0.8)
-		(drill 0.7)
+		(drill 0.6)
 		(layers "F.Cu" "B.Cu")
 		(net "+5V")
@@
 		(at 172.466 55.372)
 		(size 0.8)
-		(drill 0.7)
+		(drill 0.6)
 		(layers "F.Cu" "B.Cu")
 		(net "+5V")
@@
 		(at 159.766 55.626)
 		(size 0.8)
-		(drill 0.7)
+		(drill 0.6)
 		(layers "F.Cu" "B.Cu")
 		(net "+5V")
@@
 		(at 134.62 106.426)
 		(size 0.8)
-		(drill 0.7)
+		(drill 0.6)
 		(layers "F.Cu" "B.Cu")
 		(net "+5V")
@@
 		(at 159.512 81.026)
 		(size 0.8)
-		(drill 0.7)
+		(drill 0.6)
 		(layers "F.Cu" "B.Cu")
 		(net "+5V")
@@
 		(at 121.158 55.118)
 		(size 0.8)
-		(drill 0.7)
+		(drill 0.6)
 		(layers "F.Cu" "B.Cu")
 		(net "+5V")
