File: Hardware/PumpMotherboard/PumpMotherboard.kicad_pcb (KiCad board)
At the start: 2 copper layers, 86.4 x 91.4 mm, 63 parts, among them J1 BTB, J2 AC_LEDs, J3 T_SENSOR, J4 T_SENSOR, J401 12V Input, J5 T_SENSOR, J6 SW_IN0, J7 SW_IN1, J8 SW_IN2, M1 Fan_4pin, M2 Fan_4pin, M3 Fan_4pin, M4 Fan_4pin, M5 Fan_4pin, M6 Fan_4pin, M7 Fan_4pin, M8 Fan_4pin, Q1 MMBT3904, Q10 MMBT3904, Q2 MMBT3904, Q3 MMBT3904, Q4 MMBT3904, Q5 MMBT3904, Q6 MMBT3904, Q7 MMBT3904, Q8 MMBT3904, Q9 AO4407A, U2 AP63205WU

Commit message: Tweak board a little
Routing:
- net /TACH_2: track 50.3 -> 51.3 mm
Changed lines of the file:
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@@
-	)
-	(segment
-		(start 141.8 87.6)
-		(end 143.78 89.58)
-		(width 0.3)
-		(layer "F.Cu")
-		(net "/TACH_3")
 	)
 	(segment
@@
 	)
 	(segment
-		(start 141.8 66.025)
-		(end 141.8 87.6)
-		(width 0.3)
-		(layer "F.Cu")
-		(net "/TACH_3")
-	)
-	(segment
 		(start 138.8 63.025)
 		(end 139.375 63.6)
@@
 	)
 	(segment
+		(start 141.8 66.025)
+		(end 141.8 88.2)
+		(width 0.3)
+		(layer "F.Cu")
+		(net "/TACH_3")
+	)
+	(segment
 		(start 151.22 89.58)
 		(end 145.153898 89.58)
@@
 	)
 	(segment
-		(start 143.78 89.58)
+		(start 143.18 89.58)
 		(end 145.153898 89.58)
 		(width 0.3)
@@
 	)
 	(segment
+		(start 141.8 88.2)
+		(end 143.18 89.58)
+		(width 0.3)
+		(layer "F.Cu")
+		(net "/TACH_3")
+	)
+	(segment
 		(start 141.8 65)
 		(end 141.8 67.2)
@@
 	)
 	(segment
+		(start 142.8 76.3)
+		(end 143.38 76.88)
+		(width 0.3)
+		(layer "F.Cu")
+		(net "/TACH_1")
+	)
+	(segment
+		(start 142.8 62.5125)
+		(end 142.8 76.3)
+		(width 0.3)
+		(layer "F.Cu")
+		(net "/TACH_1")
+	)
+	(segment
 		(start 156.6 69)
 		(end 148.72 76.88)
@@
 	)
 	(segment
-		(start 142.8 62.5125)
-		(end 142.8 75.785496)
+		(start 143.38 76.88)
+		(end 145.153898 76.88)
 		(width 0.3)
 		(layer "F.Cu")
@@
 		(end 160.2 62)
 		(width 0.6)
-		(layer "F.Cu")
-		(net "/TACH_1")
-	)
-	(segment
-		(start 143.894504 76.88)
-		(end 145.153898 76.88)
-		(width 0.3)
-		(layer "F.Cu")
-		(net "/TACH_1")
-	)
-	(segment
-		(start 142.8 75.785496)
-		(end 143.894504 76.88)
-		(width 0.3)
 		(layer "F.Cu")
 		(net "/TACH_1")
@@
 	)
 	(segment
+		(start 142.3 64.7)
+		(end 142.3 80.9)
+		(width 0.3)
+		(layer "F.Cu")
+		(net "/TACH_2")
+	)
+	(segment
+		(start 166.88 71.8)
+		(end 159.6 71.8)
+		(width 0.6)
+		(layer "F.Cu")
+		(net "/TACH_2")
+	)
+	(segment
 		(start 140.8 63.2)
 		(end 142.3 64.7)
@@
 	)
 	(segment
-		(start 166.88 71.8)
-		(end 159.6 71.8)
-		(width 0.6)
-		(layer "F.Cu")
-		(net "/TACH_2")
-	)
-	(segment
-		(start 142.3 79.106102)
-		(end 145.153898 81.96)
-		(width 0.3)
-		(layer "F.Cu")
-		(net "/TACH_2")
-	)
-	(segment
 		(start 149.44 81.96)
 		(end 145.153898 81.96)
@@
 	)
 	(segment
+		(start 143.36 81.96)
+		(end 145.153898 81.96)
+		(width 0.3)
+		(layer "F.Cu")
+		(net "/TACH_2")
+	)
+	(segment
 		(start 159.6 71.8)
 		(end 149.44 81.96)
@@
 	)
 	(segment
-		(start 142.3 64.7)
-		(end 142.3 79.106102)
-		(width 0.3)
-		(layer "F.Cu")
+		(start 142.3 80.9)
+		(end 143.36 81.96)
+		(width 0.3)
+		(layer "F.Cu")

Commit message: Add PCSPKR output
Parts:
- added J9: SPKR, Connector_PinHeader_2.54mm:PinHeader_1x04_P2.54mm_Vertical, F.Cu at (109.7, 99.0)
Connections:
- A1 pad 29: unconnected-(A1-GPIO22-Pad29) -> /PCSPKR
Routing:
- net /PCSPKR: track 0.00 -> 16.8 mm, vias 0 -> 1
- net GND: vias 40 -> 39
Other:
- board text added: "SPKR"
