File: Hardware/PumpMotherboard/PumpMotherboard.kicad_pcb (KiCad board)
At the start: 2 copper layers, 86.4 x 91.4 mm, 64 parts, among them J1 BTB, J2 AC_LEDs, J3 T_SENSOR, J4 T_SENSOR, J401 12V Input, J5 T_SENSOR, J6 SW_IN0, J7 SW_IN1, J8 SW_IN2, J9 SPKR, M1 Fan_4pin, M2 Fan_4pin, M3 Fan_4pin, M4 Fan_4pin, M5 Fan_4pin, M6 Fan_4pin, M7 Fan_4pin, M8 Fan_4pin, Q1 MMBT3904, Q10 MMBT3904, Q2 MMBT3904, Q3 MMBT3904, Q4 MMBT3904, Q5 MMBT3904, Q6 MMBT3904, Q7 MMBT3904, Q8 MMBT3904, Q9 AO4407A, U2 AP63205WU

Commit message: Fix the package width for the a04407a
Parts:
- Q9: footprint Package_SO:SOIC-8_5.3x5.3mm_P1.27mm -> Package_SO:SOIC-8_3.9x4.9mm_P1.27mm
Routing:
- net +12V: track 85.8 -> 89.1 mm

Commit message: Add bulk cap
Parts:
- added C3: 10uF, Capacitor_THT:CP_Radial_D10.0mm_P5.00mm, F.Cu at (111.3, 58.0)
Routing:
- net +5V: track 118.0 -> 122.8 mm

Commit message: Add current limits for PWM in
Parts:
- added R24: 1K, Resistor_SMD:R_0805_2012Metric, F.Cu at (188.7, 93.9)
- added R25: 1K, Resistor_SMD:R_0805_2012Metric, F.Cu at (195.1, 93.9)
- added R26: 1K, Resistor_SMD:R_0805_2012Metric, F.Cu at (201.5, 88.9)
- added R27: 1K, Resistor_SMD:R_0805_2012Metric, F.Cu at (188.7, 88.9)
- added R28: 1K, Resistor_SMD:R_0805_2012Metric, F.Cu at (188.7, 84.0)
- added R29: 1K, Resistor_SMD:R_0805_2012Metric, F.Cu at (195.1, 88.9)
- added R30: 1K, Resistor_SMD:R_0805_2012Metric, F.Cu at (195.1, 84.0)
- added R31: 1K, Resistor_SMD:R_0805_2012Metric, F.Cu at (201.5, 84.0)
Connections:
- M1 pad 3: /TACH_0 -> Net-(M1-Tacho)
- M2 pad 3: /TACH_1 -> Net-(M2-Tacho)
- M3 pad 3: /TACH_2 -> Net-(M3-Tacho)
- M4 pad 3: /TACH_3 -> Net-(M4-Tacho)
- M5 pad 3: /TACH_4 -> Net-(M5-Tacho)
- M6 pad 3: /TACH_5 -> Net-(M6-Tacho)
- M7 pad 3: /TACH_6 -> Net-(M7-Tacho)
- M8 pad 3: /TACH_7 -> Net-(M8-Tacho)

Commit message: Start adding new pieces
Parts:
- added J10: USB_A, Connector_USB:USB_B_TE_5787834_Vertical, F.Cu at (133.5, 147.8)
- added U1: RP2350A, Package_DFN_QFN:QFN-60-1EP_7x7mm_P0.4mm_EP3.4x3.4mm, F.Cu at (129.0, 162.4)
