File: Hardware/PumpMotherboard/fan.kicad_sch (KiCad schematic)
At the start: 4 parts, among them M1 Fan_4pin, Q1 MMBT3904

Commit message: Add LCSC part num
Parts:
- M1: LCSC# (none) -> C240840
Changed lines of the file:
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@@
+			)
+		)
+		(property "LCSC#" "C240840"
+			(at 156.21 101.6 0)
+			(hide yes)
+			(show_name no)
+			(do_not_autoplace no)
+			(effects
+				(font
+					(size 1.27 1.27)
+				)
 			)
 		)

Commit message: Add 12v power switching
Connections:
- net +12V renamed 12V_SWITCHED
Changed lines of the file:
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@@
 	(wire
 		(pts
-			(xy 156.21 91.44) (xy 156.21 93.98)
+			(xy 156.21 90.17) (xy 156.21 93.98)
 		)
 		(stroke
@@
 	(wire
 		(pts
-			(xy 138.43 92.71) (xy 138.43 91.44)
+			(xy 158.75 90.17) (xy 156.21 90.17)
 		)
 		(stroke
@@
 	(wire
 		(pts
-			(xy 156.21 106.68) (xy 156.21 119.38)
+			(xy 138.43 92.71) (xy 138.43 91.44)
 		)
 		(stroke
@@
 	(wire
 		(pts
-			(xy 113.03 111.76) (xy 116.84 111.76)
+			(xy 156.21 106.68) (xy 156.21 119.38)
 		)
 		(stroke
@@
 	(wire
 		(pts
-			(xy 138.43 116.84) (xy 138.43 119.38)
+			(xy 113.03 111.76) (xy 116.84 111.76)
 		)
 		(stroke
@@
 	(wire
 		(pts
-			(xy 121.92 111.76) (xy 130.81 111.76)
+			(xy 138.43 116.84) (xy 138.43 119.38)
 		)
 		(stroke
 			(width 0)
 			(type default)
+		)
+	)
+	(wire
+		(pts
+			(xy 121.92 111.76) (xy 130.81 111.76)
+		)
+		(stroke
+			(width 0)
+			(type default)
+		)
+	)
+	(global_label "12V_SWITCHED"
+		(shape input)
+		(at 158.75 90.17 0)
+		(fields_autoplaced yes)
+		(effects
+			(font
+				(size 1.27 1.27)
+			)
+			(justify left)
+		)
+		(property "Intersheetrefs" "${INTERSHEET_REFS}"
+			(at 175.4632 90.17 0)
+			(hide yes)
+			(show_name no)
+			(do_not_autoplace no)
+			(effects
+				(font
+					(size 1.27 1.27)
+				)
+				(justify left)
+			)
 		)
 	)
@@
 					(unit 1)
 				)
-			)
-		)
-	)
-	(symbol
-		(lib_id "power:+12V")
-		(at 156.21 91.44 0)
-		(unit 1)
-		(body_style 1)
-		(exclude_from_sim no)
-		(in_bom yes)
-		(on_board yes)
-		(in_pos_files yes)
-		(dnp no)
-		(fields_autoplaced yes)
-		(property "Reference" "#PWR01"
-			(at 156.21 95.25 0)
-			(hide yes)
-			(show_name no)
-			(do_not_autoplace no)
-			(effects
-				(font
-					(size 1.27 1.27)
-				)
-			)
-		)
-		(property "Value" "+12V"
-			(at 156.21 86.36 0)
-			(show_name no)
-			(do_not_autoplace no)
-			(effects
-				(font
-					(size 1.27 1.27)
-				)
-			)
-		)
-		(property "Footprint" ""
-			(at 156.21 91.44 0)
-			(hide yes)
-			(show_name no)
-			(do_not_autoplace no)
-			(effects
-				(font
-					(size 1.27 1.27)
-				)
-			)
-		)
-		(property "Datasheet" ""
-			(at 156.21 91.44 0)
-			(hide yes)
-			(show_name no)
-			(do_not_autoplace no)
-			(effects
-				(font
-					(size 1.27 1.27)
-				)
-			)
-		)
-		(property "Description" "Power symbol creates a global label with name \"+12V\""
-			(at 156.21 91.44 0)
-			(hide yes)
-			(show_name no)
-			(do_not_autoplace no)
-			(effects
-				(font
-					(size 1.27 1.27)
-				)
-			)
-		)
-		(pin "1"
-		)
-		(instances
-			(project "PumpMotherboard"
-				(path "/0d3b5c69-c1f2-4eab-9f51-de1d9dac9894/2e044f8d-c712-4cd3-88f5-f08c3236630a"
-					(reference "#PWR014")
-					(unit 1)
-				)
-				(path "/0d3b5c69-c1f2-4eab-9f51-de1d9dac9894/2e552afc-dcec-4b80-9f54-686ad7c15326"
-					(reference "#PWR011")
-					(unit 1)
-				)
-				(path "/0d3b5c69-c1f2-4eab-9f51-de1d9dac9894/4b5fcaae-9e0c-4939-99e5-bcb8dde5d82b"
-					(reference "#PWR01")
-					(unit 1)
-				)
-				(path "/0d3b5c69-c1f2-4eab-9f51-de1d9dac9894/6a4583d5-71e1-4585-bb00-68155c4aeca7"
-					(reference "#PWR033")
-					(unit 1)
-				)
-				(path "/0d3b5c69-c1f2-4eab-9f51-de1d9dac9894/7a92dd86-2d0d-4c0b-841e-dcdaa321ed19"
-					(reference "#PWR037")
-					(unit 1)
-				)
-				(path "/0d3b5c69-c1f2-4eab-9f51-de1d9dac9894/941dab02-31b2-4d8d-a9b2-b16910241135"
-					(reference "#PWR029")
-					(unit 1)
-				)
-				(path "/0d3b5c69-c1f2-4eab-9f51-de1d9dac9894/b498c0a6-5114-4fdb-8c71-abd72c5fb2ff"
-					(reference "#PWR05")
-					(unit 1)
-				)
-				(path "/0d3b5c69-c1f2-4eab-9f51-de1d9dac9894/ed796959-e196-4a03-9c52-bbbb27f18f72"
-					(reference "#PWR08")
-					(unit 1)
-				)

Commit message: Add current limits for PWM in
Parts:
- added R24: 1K, Resistor_SMD:R_0805_2012Metric, symbol Device:R_Small
Connections:
- net TACH_OUT: now also R24.1; no longer M1.3 (Tacho)
- new net: M1.3 (Tacho), R24.2
Other:
- moved on the sheet: R1
Changed lines of the file:
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@@
 	(paper "A4")
 	(junction
-		(at 138.43 99.06)
+		(at 124.46 99.06)
 		(diameter 0)
 		(color 0 0 0 0)
@@
 	(wire
 		(pts
-			(xy 113.03 99.06) (xy 138.43 99.06)
-		)
-		(stroke
-			(width 0)
-			(type default)
-		)
-	)
-	(wire
-		(pts
-			(xy 138.43 97.79) (xy 138.43 99.06)
+			(xy 113.03 99.06) (xy 135.89 99.06)
+		)
+		(stroke
+			(width 0)
+			(type default)
+		)
+	)
+	(wire
+		(pts
+			(xy 124.46 97.79) (xy 124.46 99.06)
 		)
 		(stroke
@@
 	(wire
 		(pts
-			(xy 138.43 99.06) (xy 148.59 99.06)
-		)
-		(stroke
-			(width 0)
-			(type default)
-		)
-	)
-	(wire
-		(pts
 			(xy 156.21 90.17) (xy 156.21 93.98)
 		)
@@
 	(wire
 		(pts
-			(xy 138.43 92.71) (xy 138.43 91.44)
+			(xy 124.46 92.71) (xy 124.46 91.44)
 		)
 		(stroke
@@
 		(pts
 			(xy 156.21 106.68) (xy 156.21 119.38)
+		)
+		(stroke
+			(width 0)
+			(type default)
+		)
+	)
+	(wire
+		(pts
+			(xy 140.97 99.06) (xy 148.59 99.06)
 		)
 		(stroke
@@
 	(symbol
 		(lib_id "power:+3V3")
-		(at 138.43 91.44 0)
+		(at 124.46 91.44 0)
 		(unit 1)
 		(body_style 1)
@@
 		(fields_autoplaced yes)
 		(property "Reference" "#PWR023"
-			(at 138.43 95.25 0)
+			(at 124.46 95.25 0)
 			(hide yes)
 			(show_name no)
@@
 		)
 		(property "Value" "+3V3"
-			(at 138.43 86.36 0)
+			(at 124.46 86.36 0)
 			(show_name no)
 			(do_not_autoplace no)
@@
 		)
 		(property "Footprint" ""
-			(at 138.43 91.44 0)
+			(at 124.46 91.44 0)
 			(hide yes)
 			(show_name no)
@@
 		)
 		(property "Datasheet" ""
-			(at 138.43 91.44 0)
+			(at 124.46 91.44 0)
 			(hide yes)
 			(show_name no)
@@
 		)
 		(property "Description" "Power symbol creates a global label with name \"+3V3\""
-			(at 138.43 91.44 0)
+			(at 124.46 91.44 0)
 			(hide yes)
 			(show_name no)
@@
 	(symbol
 		(lib_id "Device:R_Small")
-		(at 138.43 95.25 0)
+		(at 124.46 95.25 0)
 		(unit 1)
 		(body_style 1)
@@
 		(fields_autoplaced yes)
 		(property "Reference" "R1"
-			(at 140.97 93.9799 0)
+			(at 127 93.9799 0)
 			(show_name no)
 			(do_not_autoplace no)
@@
 		)
 		(property "Value" "10K"
-			(at 140.97 96.5199 0)
+			(at 127 96.5199 0)
 			(show_name no)
 			(do_not_autoplace no)
@@
 		)
 		(property "Footprint" "Resistor_SMD:R_0805_2012Metric"
-			(at 138.43 95.25 0)
+			(at 124.46 95.25 0)
 			(hide yes)
 			(show_name no)
@@
 		)
 		(property "Datasheet" ""
-			(at 138.43 95.25 0)
+			(at 124.46 95.25 0)
 			(hide yes)
 			(show_name no)
@@
 		)
 		(property "Description" "Resistor, small symbol"
-			(at 138.43 95.25 0)
+			(at 124.46 95.25 0)
 			(hide yes)
 			(show_name no)
@@
 					(unit 1)
 				)
+			)
+		)
+	)
+	(symbol
+		(lib_id "Device:R_Small")
+		(at 138.43 99.06 90)
+		(unit 1)
+		(body_style 1)
+		(exclude_from_sim no)
+		(in_bom yes)
+		(on_board yes)
+		(in_pos_files yes)
+		(dnp no)
+		(fields_autoplaced yes)
+		(property "Reference" "R24"
+			(at 138.43 93.98 90)
+			(show_name no)
+			(do_not_autoplace no)
+			(effects
+				(font
+					(size 1.016 1.016)
+				)
+			)
+		)
+		(property "Value" "1K"
+			(at 138.43 96.52 90)
+			(show_name no)
+			(do_not_autoplace no)
+			(effects
+				(font
+					(size 1.27 1.27)
+				)
+			)
+		)
+		(property "Footprint" "Resistor_SMD:R_0805_2012Metric"
+			(at 138.43 99.06 0)
+			(hide yes)
+			(show_name no)
+			(do_not_autoplace no)
+			(effects
+				(font
+					(size 1.27 1.27)
+				)
+			)
+		)
+		(property "Datasheet" ""
+			(at 138.43 99.06 0)
+			(hide yes)
+			(show_name no)
+			(do_not_autoplace no)
+			(effects
+				(font
+					(size 1.27 1.27)
+				)
+			)
+		)
+		(property "Description" "Resistor, small symbol"
+			(at 138.43 99.06 0)
+			(hide yes)
+			(show_name no)
+			(do_not_autoplace no)
+			(effects
+				(font
+					(size 1.27 1.27)
+				)
+			)
+		)
+		(pin "2"
+		)
+		(pin "1"
+		)
+		(instances
+			(project "PumpMotherboard"
+				(path "/0d3b5c69-c1f2-4eab-9f51-de1d9dac9894/2e044f8d-c712-4cd3-88f5-f08c3236630a"
+					(reference "R28")
+					(unit 1)
+				)
+				(path "/0d3b5c69-c1f2-4eab-9f51-de1d9dac9894/2e552afc-dcec-4b80-9f54-686ad7c15326"
+					(reference "R27")
+					(unit 1)
+				)
+				(path "/0d3b5c69-c1f2-4eab-9f51-de1d9dac9894/4b5fcaae-9e0c-4939-99e5-bcb8dde5d82b"
+					(reference "R24")
+					(unit 1)
+				)
+				(path "/0d3b5c69-c1f2-4eab-9f51-de1d9dac9894/6a4583d5-71e1-4585-bb00-68155c4aeca7"
+					(reference "R30")
+					(unit 1)
+				)
+				(path "/0d3b5c69-c1f2-4eab-9f51-de1d9dac9894/7a92dd86-2d0d-4c0b-841e-dcdaa321ed19"
+					(reference "R31")
+					(unit 1)
+				)
+				(path "/0d3b5c69-c1f2-4eab-9f51-de1d9dac9894/941dab02-31b2-4d8d-a9b2-b16910241135"
+					(reference "R29")
+					(unit 1)
+				)
+				(path "/0d3b5c69-c1f2-4eab-9f51-de1d9dac9894/b498c0a6-5114-4fdb-8c71-abd72c5fb2ff"
+					(reference "R25")
+					(unit 1)
+				)
+				(path "/0d3b5c69-c1f2-4eab-9f51-de1d9dac9894/ed796959-e196-4a03-9c52-bbbb27f18f72"
+					(reference "R26")
+					(unit 1)
+				)
